Commit message: added a program fruit_ninja that will be used to perform ikin on the robot

File: project_ws/src/fruitninja/urdf/fruitNinja.urdf (robot description, URDF)
Before this commit: robot FruitNinja, 28 links, 27 joints
Joints:
- joint final: origin xyz=0 0.15 0 rpy=1.5708 0 3.1416 -> xyz=0 0.3 0 rpy=0 0 0
