Commit message: Added sabre to URDF

File: fruitNinja.urdf (robot description, URDF)
Before this commit: robot FruitNinja, 28 links, 27 joints
Links:
- removed link katana
- added link sabre, mass 0.60441; collision mesh filename=package://Sabre/meshes/Sabre.STL; visual mesh filename=package://Sabre/meshes/Sabre.STL
Joints:
- removed joint attach-katana
- added joint attach-sabre: type fixed, parent link7, child sabre

File: project_ws/src/fruitninja/urdf/fruitNinja.urdf (robot description, URDF)
Before this commit: robot FruitNinja, 28 links, 27 joints
Links:
- removed link katana
- added link sabre, mass 0.60441; collision mesh filename=package://Sabre/meshes/Sabre.STL; visual mesh filename=package://Sabre/meshes/Sabre.STL
Joints:
- removed joint attach-katana
- added joint attach-sabre: type fixed, parent link7, child sabre
- joint final: origin xyz=0 0.3 0 rpy=0 0 0 -> xyz=0 0.15 0 rpy=1.5708 0 3.1416
